File: sord-m5-romcart.kicad_pcb (KiCad board)
At the start: 2 copper layers, 1 part, among them U2 27C256

Commit message: Board outline
Parts:
- added U1: ~, Sord:M5_CartridgeSlot, F.Cu at (189.2, 152.9)
- U2: moved to B.Cu
- moved U2 127.1 mm to (172.5, 133.9)
Other:
- board outline added: 101.1 x 62.5 mm

Commit message: Symbol cleanout
Connections:
- U1 pad A1: (no net) -> -12V
- U1 pad A10: (no net) -> /D1
- U1 pad A11: (no net) -> /D0
- U1 pad A12: (no net) -> /A7
- U1 pad A13: (no net) -> /A6
- U1 pad A14: (no net) -> /A5
- U1 pad A15: (no net) -> /A4
- U1 pad A16: (no net) -> /A3
- U1 pad A17: (no net) -> /A2
- U1 pad A18: (no net) -> /A1
- U1 pad A19: (no net) -> /A0
- U1 pad A2: (no net) -> +12V
- U1 pad A20: (no net) -> unconnected-(U1-~{WAIT}-PadA20)
- U1 pad A21: (no net) -> unconnected-(U1-~{ROMDS}-PadA21)
- U1 pad A22: (no net) -> /~{ROM0}
- U1 pad A23: (no net) -> unconnected-(U1-~{ROM2}-PadA23)
- U1 pad A24: (no net) -> /~{MEM_RD}
- U1 pad A25: (no net) -> unconnected-(U1-~{IO_RD}-PadA25)
- U1 pad A26: (no net) -> unconnected-(U1-~{EX_IOA}-PadA26)
- U1 pad A27: (no net) -> unconnected-(U1-~{EX_INT}-PadA27)
- U1 pad A28: (no net) -> unconnected-(U1-~{RESET}-PadA28)
- U1 pad A3: (no net) -> +12V
- U1 pad A4: (no net) -> +5V
- U1 pad A5: (no net) -> +5V
- U1 pad A6: (no net) -> GND
- U1 pad A7: (no net) -> GND
- U1 pad A8: (no net) -> /D3
- U1 pad A9: (no net) -> /D2
- U1 pad B1: (no net) -> -12V
- U1 pad B10: (no net) -> /D6
- U1 pad B11: (no net) -> /D7
- U1 pad B12: (no net) -> /A8
- U1 pad B13: (no net) -> /A9
- U1 pad B14: (no net) -> /A10
- U1 pad B15: (no net) -> /A11
- U1 pad B16: (no net) -> /A12
- U1 pad B17: (no net) -> unconnected-(U1-A13-PadB17)
- U1 pad B18: (no net) -> unconnected-(U1-A14-PadB18)
- U1 pad B19: (no net) -> unconnected-(U1-A15-PadB19)
- U1 pad B2: (no net) -> +12V
- U1 pad B20: (no net) -> unconnected-(U1-~{MEMRQ}-PadB20)
- U1 pad B21: (no net) -> unconnected-(U1-~{RFSH}-PadB21)
- U1 pad B22: (no net) -> /~{ROM1}
- U1 pad B23: (no net) -> unconnected-(U1-~{EXM}-PadB23)
- U1 pad B24: (no net) -> unconnected-(U1-~{MEM_WR}-PadB24)
- U1 pad B25: (no net) -> unconnected-(U1-~{IO_WR}-PadB25)
- U1 pad B26: (no net) -> unconnected-(U1-~{EX_IOB}-PadB26)
- U1 pad B27: (no net) -> unconnected-(U1-EX_CLK-PadB27)
- U1 pad B28: (no net) -> unconnected-(U1-CLK-PadB28)
- U1 pad B3: (no net) -> +12V
- U1 pad B4: (no net) -> +5V
- U1 pad B5: (no net) -> +5V
- U1 pad B6: (no net) -> GND
- U1 pad B7: (no net) -> GND
- U1 pad B8: (no net) -> /D4
- U1 pad B9: (no net) -> /D5

Commit message: Significant symbol mess
Routing:
- net GND: track 0.00 -> 42.4 mm, vias 0 -> 4
- net +5V: track 0.00 -> 27.2 mm, vias 0 -> 2
- net +12V: track 0.00 -> 27.2 mm, vias 0 -> 2
Changed lines of the file:
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@@
 		)
+	)
+	(segment
+		(start 179.07 148.0185)
+		(end 179.07 137.414)
+		(width 1)
+		(layer "F.Cu")
+		(net 2)
+	)
+	(segment
+		(start 176.53 148.0185)
+		(end 176.53 137.414)
+		(width 1)
+		(layer "F.Cu")
+		(net 2)
+	)
+	(via
+		(at 176.53 141.732)
+		(size 0.6)
+		(drill 0.3)
+		(layers "F.Cu" "B.Cu")
+		(net 2)
+	)
+	(via
+		(at 179.07 141.732)
+		(size 0.6)
+		(drill 0.3)
+		(layers "F.Cu" "B.Cu")
+		(net 2)
+	)
+	(via
+		(at 179.07 137.414)
+		(size 0.6)
+		(drill 0.3)
+		(layers "F.Cu" "B.Cu")
+		(net 2)
+	)
+	(via
+		(at 176.53 137.414)
+		(size 0.6)
+		(drill 0.3)
+		(layers "F.Cu" "B.Cu")
+		(net 2)
+	)
+	(segment
+		(start 176.53 148.0185)
+		(end 176.53 141.732)
+		(width 1)
+		(layer "B.Cu")
+		(net 2)
+	)
+	(segment
+		(start 179.07 148.0185)
+		(end 179.07 141.732)
+		(width 1)
+		(layer "B.Cu")
+		(net 2)
+	)
+	(segment
+		(start 179.07 141.732)
+		(end 179.07 137.414)
+		(width 1)
+		(layer "B.Cu")
+		(net 2)
+	)
+	(segment
+		(start 176.53 141.732)
+		(end 176.53 137.414)
+		(width 1)
+		(layer "B.Cu")
+		(net 2)
+	)
+	(segment
+		(start 181.61 142.494)
+		(end 181.61 148.0185)
+		(width 1)
+		(layer "F.Cu")
+		(net 10)
+	)
+	(segment
+		(start 184.15 148.0185)
+		(end 184.15 142.494)
+		(width 1)
+		(layer "F.Cu")
+		(net 10)
+	)
+	(segment
+		(start 184.15 142.494)
+		(end 181.61 142.494)
+		(width 1)
+		(layer "F.Cu")
+		(net 10)
+	)
+	(via
+		(at 184.15 142.494)
+		(size 0.6)
+		(drill 0.3)
+		(layers "F.Cu" "B.Cu")
+		(net 10)
+	)
+	(via
+		(at 181.61 142.494)
+		(size 0.6)
+		(drill 0.3)
+		(layers "F.Cu" "B.Cu")
+		(net 10)
+	)
+	(segment
+		(start 184.15 142.494)
+		(end 181.61 142.494)
+		(width 1)
+		(layer "B.Cu")
+		(net 10)
+	)
+	(segment
+		(start 184.15 148.0185)
+		(end 184.15 142.494)
+		(width 1)
+		(layer "B.Cu")
+		(net 10)
+	)
+	(segment
+		(start 181.61 142.494)
+		(end 181.61 148.0185)
+		(width 1)
+		(layer "B.Cu")
+		(net 10)
+	)
+	(segment
+		(start 189.23 148.0185)
+		(end 189.23 142.494)
+		(width 1)
+		(layer "F.Cu")
+		(net 35)
+	)
+	(segment
+		(start 186.69 142.494)
+		(end 186.69 148.0185)
+		(width 1)
+		(layer "F.Cu")
+		(net 35)
+	)
+	(segment
+		(start 189.23 142.494)
+		(end 186.69 142.494)
+		(width 1)
+		(layer "F.Cu")
+		(net 35)
+	)
+	(via
+		(at 189.23 142.494)
+		(size 0.6)
+		(drill 0.3)
+		(layers "F.Cu" "B.Cu")
+		(net 35)
+	)
+	(via
+		(at 186.69 142.494)
+		(size 0.6)
+		(drill 0.3)
+		(layers "F.Cu" "B.Cu")
+		(net 35)
+	)
+	(segment
+		(start 189.23 148.0185)
+		(end 189.23 142.494)
+		(width 1)
+		(layer "B.Cu")
+		(net 35)
+	)
+	(segment
+		(start 189.23 142.494)
+		(end 186.69 142.494)
+		(width 1)
+		(layer "B.Cu")
+		(net 35)
+	)
+	(segment
+		(start 186.69 142.494)
+		(end 186.69 148.0185)
+		(width 1)
+		(layer "B.Cu")
+		(net 35)
 	)
 	(embedded_fonts no)

Commit message: Version numbers
Other:
- outline, holes or cut-outs redrawn
- board text added: "A1"
- board text added: "A28"
- board text added: "B1"
- board text added: "B28"
- board text added: "Parts Side"
- board text added: "Solder Side"
- board text added: "Sord M5 Prototyping/ROM board leadedsolder.com v1 2025"
Changed lines of the file:
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@@
 		(layer "Edge.Cuts")
 	)
+	(gr_circle
+		(center 196.088 138.938)
+		(end 197.612 140.462)
+		(stroke
+			(width 0.05)
+			(type default)
+		)
+		(fill no)
+		(layer "Edge.Cuts")
+	)
 	(gr_line
 		(start 199.898 140.716)
@@
 		(layer "Edge.Cuts")
 	)
+	(gr_circle
+		(center 102.87 139.192)
+		(end 104.14 140.97)
+		(stroke
+			(width 0.05)
+			(type default)
+		)
+		(fill no)
+		(layer "Edge.Cuts")
+	)
 	(gr_line
 		(start 194.31 142.494)
@@
 			"AAAAAAAAAAAAAAAAAAAAAAAAAAAAAAAAAAAAAAAAAAAAAAAAAAAAAAAAAAAAAAAAAAAAAAAAAAAA"
 			"AAAAAAAAAAAAAAAAAAAAAAAAAAAAAAAAAAAAAAAAAAAAAAAAAAAAAAAAAAAAAAAAAAAAAAAAAAAA"
+			"AAAAAAAAAAAAAAAAAAAAAAAAAAAAAAAAAAAAAAAAAAAAAAAAAAAAAAAAAAAAAAAAAAAAAAAAAAAA"
+			"AAAAAAAAAAAAAAAAAAAAAAAAAAAAAAAAAAAAAAAAAAAAAAAAAAAAAAAAAAAAAAAAAAAAAAAAAAAA"
+			"AAAAAAAAAAAAAAAAAAAAAAAAAAAAAAAAAAAAAAAAAAAAAAAAAAAAAAAAAAAAAAAAAAAAAAAAAAAA"
+			"AAAAAAAAAAAAAAAAAAAAAAAAAAAAAAAAAAAAAAAAAAAAAAAAAAAAAAAAAAAAAAAAAAAAAAAAAAAA"
+			"AAAAAAAAAAAAAAAAAAAAAAAAAAAAAAAAAAAAAAAAAAAAAAAAAAAAAAAAAAAAAAAAAAAAAAAAAAAA"
+			"AAAAAAAAAAAAAAAAAAAAAAAAAAAAAAAAAAAAAAAAAAAAAAAAAAAAAAAAAAAAAAAAAAAAAAAAAAAA"
+			"AAAAAAAAAAAAAAAAAAAAAAAAAAAAAAAAAAAAAAAAAAAAAAAAAAAAAAAAAAAAAAAAAAAAAAAAAAAA"
+			"AAAAAAAAAAAAAAAAAAAAAAAAAAAAAAAAAAAAAAAAAAAAAAAAAAAAAAAAAAAAAAAAAAAAAAAAAAAA"
+			"AAAAAAAAAAAAAAAAAAAAAAAAAAAAAAAAAAAAAAAAAAAAAAAAAAAAAAAAAAAAAAAAAAAAAAAAAAAA"
+			"AAAAAAAAAAAAAAAAAAAAAAAAAAAAAAAAAAAAAAAAAAAAAAAAAAAAAAAAAAAAAAAAAAAAAAAAAAAA"
+			"AAAAAAAAAAAAAAAAAAAAAAAAAAAAAAAAAAAAAAAAAAAAAAAAAAAAAAAAAAAAAAAAAAAAAAAAAAAA"
+			"AAAAAAAAAAAAAAAAAAAAAAAAAAAAAAAAAAAAAAAAAAAAAAAAAAAAAAAAAAAAAAAAAAAAAAAAAAAA"
+			"AAAAAAAAAAAAAAAAAAAAAAAAAAAAAAAAAAAAAAAAAAAAAAAAAAAAAAAAAAAAAAAAAAAAAAAAAAAA"
+			"AAAAAAAAAAAAAAAAAAAAAAAAAAAAAAAAAAAAAAAAAAAAAAAAAAAAAAAAAAAAAAAAAAAAAAAAAAAA"
+			"AAAAAAAAAAAAAAAAAAAAAAAAAAAAAAAAAAAAAAAAAAAAAAAAAAAAAAAAAAAAAAAAAAAAAAAAAAAA"
+			"AAAAAAAAAAAAAAAAAAAAAAAAAAAAAAAAAAAAAAAAAAAAAAAAAAAAAAAAAAAAAAAAAAAAAAAAAAAA"
+			"AAAAAAAAAAAAAAAAAAAAAAAAAAAAAAAAAAAAAAAAAAAAAAAAAAAAAAAAAAAAAAAAAAAAAAAAAAAA"
+			"AAAAAAAAAAAAAAAAAAAAAAAAAAAAAAAAAAAAAAAAAAAAAAAAAAAAAAAAAAAAAAAAAAAAAAAAAAAA"
 			"AAAAAAAAAAAAAA=="
 		)
 	)
+	(gr_text "Sord M5 Prototyping/ROM board\nleadedsolder.com v1 2025"
+		(at 106.934 140.97 0)
+		(layer "F.SilkS")
+		(effects
+			(font
+				(size 1 1)
+				(thickness 0.1)
+			)
+			(justify left bottom)
+		)
+	)
+	(gr_text "Solder Side"
+		(at 101.092 94.234 0)
+		(layer "F.SilkS")
+		(effects
+			(font
+				(size 1 1)
+				(thickness 0.1)
+			)
+			(justify left bottom)
+		)
+	)
+	(gr_text "A28"
+		(at 121.759048 142.748 0)
+		(layer "F.SilkS")
+		(effects
+			(font
+				(size 1 1)
+				(thickness 0.1)
+			)
+			(justify left bottom)
+		)
+	)
+	(gr_text "A1"
+		(at 190.815238 142.748 0)
+		(layer "F.SilkS")
+		(effects
+			(font
+				(size 1 1)
+				(thickness 0.1)
+			)
+			(justify left bottom)
+		)
+	)
+	(gr_text "B1"
+		(at 192.796191 142.748 0)
+		(layer "B.SilkS")
+		(effects
+			(font
+				(size 1 1)
+				(thickness 0.1)
+			)
+			(justify left bottom mirror)
+		)
+	)
+	(gr_text "Parts Side"
+		(at 109.22 94.234 0)
+		(layer "B.SilkS")
+		(effects
+			(font
+				(size 1 1)
+				(thickness 0.1)
+			)
+			(justify left bottom mirror)
+		)
+	)
+	(gr_text "B28"
+		(at 124.714 142.748 0)
+		(layer "B.SilkS")
+		(effects
+			(font
+				(size 1 1)
+				(thickness 0.1)
+			)
+			(justify left bottom mirror)
+		)
+	)

Commit message: V1 sent to fab
Parts:
- added R1: 10kΩ, Resistor_THT:R_Axial_DIN0207_L6.3mm_D2.5mm_P10.16mm_Horizontal, B.Cu at (192.4, 131.4)
- added REF**: Prototyping_Area, Sord:Prototyping_Area, B.Cu at (130.2, 116.2)
- added SW1: Choose ROM, Connector_PinHeader_2.54mm:PinHeader_1x02_P2.54mm_Vertical, B.Cu at (192.4, 116.2)
- added U3: 74LS00, Package_DIP:DIP-14_W7.62mm_Socket_LongPads, B.Cu at (154.3, 115.8)
- U2: footprint Package_DIP:DIP-28_W15.24mm -> Package_DIP:DIP-28_W15.24mm_Socket_LongPads
Connections:
- U1 pad A23: unconnected-(U1-~{ROM2}-PadA23) -> /~{ROM2}
- U2 pad 20: /~{ROM0} -> /~{ROM_CS}
- U2 pad 26: unconnected-(U2-A13-Pad26) -> /ROM_A13
- U2 pad 27: unconnected-(U2-A14-Pad27) -> /ROM_A14
Routing:
- net /~{MEM_RD}: track 0.00 -> 84.6 mm, vias 0 -> 3
- net /~{ROM1}: track 0.00 -> 69.2 mm, vias 0 -> 5
- net /A0: track 0.00 -> 66.8 mm, vias 0 -> 3
- net /D7: track 0.00 -> 61.6 mm, vias 0 -> 2
- net /A10: track 0.00 -> 61.5 mm, vias 0 -> 2
- net /A1: track 0.00 -> 60.9 mm, vias 0 -> 1
- net /D3: track 0.00 -> 60.5 mm, vias 0 -> 1
- net /D6: track 0.00 -> 60.1 mm, vias 0 -> 4
- net /A11: track 0.00 -> 60.1 mm, vias 0 -> 4
- net /D5: track 0.00 -> 59.3 mm, vias 0 -> 2
- net /D4: track 0.00 -> 57.5 mm, vias 0 -> 2
- net /A2: track 0.00 -> 55.8 mm, vias 0 -> 1
- net /ROM_A13: track 0.00 -> 55.0 mm, vias 0 -> 2
- net /A9: track 0.00 -> 54.1 mm, vias 0 -> 2
- net /A8: track 0.00 -> 49.1 mm, vias 0 -> 2
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- added copper zone on B.Cu, net +5V
- added copper zone on F.Cu, net GND
Other:
- board size 101.1 x 62.5 mm -> 99.3 x 62.5 mm
- board text added: "+5V"
- board text added: "1"
- board text added: "10"
- board text added: "11"
- board text added: "12"
- board text added: "2"
- board text added: "3"
- board text added: "4"
- board text added: "5"
- board text added: "6"
- board text added: "7"
- board text added: "8"
- board text added: "9"
- board text added: "A"
- board text added: "B"
- board text added: "C"
- board text added: "D"
- board text added: "E"
- board text added: "F"
- board text added: "G"
- board text added: "GND"
- board text added: "H"
- board text added: "I"
- board text added: "J"
- board text added: "K"
- board text added: "L"

Commit message: Use hole footprints for the sake of TurboCase later
Parts:
- added REF**: MountingHole_3.2mm_M3, MountingHole:MountingHole_3.2mm_M3, F.Cu at (196.1, 138.9)
- added REF**: MountingHole_3.2mm_M3, MountingHole:MountingHole_3.2mm_M3, F.Cu at (104.1, 139.2)
Other:
- outline, holes or cut-outs redrawn
- board text added: "Sord M5 Prototyping/ROM board leadedsolder.com v2 2025"
- board text removed: "Sord M5 Prototyping/ROM board leadedsolder.com v1 2025"
Changed lines of the file:
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@@
 	(net 50 "unconnected-(U3-Pad11)")
 	(net 51 "Net-(U3-Pad3)")
+	(footprint "MountingHole:MountingHole_3.2mm_M3"
+		(locked yes)
+		(layer "F.Cu")
+		(at 196.088 138.938)
+		(descr "Mounting Hole 3.2mm, no annular, M3")
+		(tags "mounting hole 3.2mm no annular m3")
+		(property "Reference" "REF**"
+			(at 0 -4.2 0)
+			(layer "F.SilkS")
+			(hide yes)
+			(effects
+				(font
+					(size 1 1)
+					(thickness 0.15)
+				)
+			)
+		)
+		(property "Value" "MountingHole_3.2mm_M3"
+			(at 0 4.2 0)
+			(layer "F.Fab")
+			(effects
+				(font
+					(size 1 1)
+					(thickness 0.15)
+				)
+			)
+		)
+		(property "Datasheet" ""
+			(at 0 0 0)
+			(unlocked yes)
+			(layer "F.Fab")
+			(hide yes)
+			(effects
+				(font
+					(size 1.27 1.27)
+					(thickness 0.15)
+				)
+			)
+		)
+		(property "Description" ""
+			(at 0 0 0)
+			(unlocked yes)
+			(layer "F.Fab")
+			(hide yes)
+			(effects
+				(font
+					(size 1.27 1.27)
+					(thickness 0.15)
+				)
+			)
+		)
+		(attr board_only exclude_from_pos_files exclude_from_bom dnp)
+		(fp_circle
+			(center 0 0)
+			(end 3.2 0)
+			(stroke
+				(width 0.15)
+				(type solid)
+			)
+			(fill no)
+			(layer "Cmts.User")
+		)
+		(fp_circle
+			(center 0 0)
+			(end 3.45 0)
+			(stroke
+				(width 0.05)
+				(type solid)
+			)
+			(fill no)
+			(layer "F.CrtYd")
+		)
+		(fp_text user "${REFERENCE}"
+			(at 0 0 0)
+			(layer "F.Fab")
+			(effects
+				(font
+					(size 1 1)
+					(thickness 0.15)
+				)
+			)
+		)
+		(pad "" np_thru_hole circle
+			(at 0 0)
+			(size 3.2 3.2)
+			(drill 3.2)
+			(layers "*.Cu" "*.Mask")
+		)
+		(embedded_fonts no)
+	)
 	(footprint "Sord:M5_CartridgeSlot"
 		(layer "F.Cu")
@@
 		(embedded_fonts no)
 	)
+	(footprint "MountingHole:MountingHole_3.2mm_M3"
+		(locked yes)
+		(layer "F.Cu")
+		(at 104.14 139.192)
+		(descr "Mounting Hole 3.2mm, no annular, M3")
+		(tags "mounting hole 3.2mm no annular m3")
+		(property "Reference" "REF**"
+			(at 0 -4.2 0)
+			(layer "F.SilkS")
+			(hide yes)
+			(effects
+				(font
+					(size 1 1)
+					(thickness 0.15)
+				)
+			)
+		)
+		(property "Value" "MountingHole_3.2mm_M3"
+			(at 0 4.2 0)
+			(layer "F.Fab")
+			(effects
+				(font
+					(size 1 1)
+					(thickness 0.15)
+				)
+			)
+		)
+		(property "Datasheet" ""
+			(at 0 0 0)
+			(unlocked yes)
+			(layer "F.Fab")
+			(hide yes)
+			(effects
+				(font
+					(size 1.27 1.27)
+					(thickness 0.15)
+				)
+			)
+		)
+		(property "Description" ""
+			(at 0 0 0)
+			(unlocked yes)
+			(layer "F.Fab")
+			(hide yes)
+			(effects
+				(font
+					(size 1.27 1.27)
+					(thickness 0.15)
+				)
+			)
+		)
+		(attr board_only exclude_from_pos_files exclude_from_bom dnp)
+		(fp_circle
+			(center 0 0)
+			(end 3.2 0)
+			(stroke
+				(width 0.15)
+				(type solid)
+			)
+			(fill no)
+			(layer "Cmts.User")
+		)
+		(fp_circle
+			(center 0 0)
+			(end 3.45 0)
+			(stroke
+				(width 0.05)
+				(type solid)
+			)
+			(fill no)
+			(layer "F.CrtYd")
+		)
+		(fp_text user "${REFERENCE}"
+			(at 0 0 0)
+			(layer "F.Fab")
+			(effects
+				(font
+					(size 1 1)
+					(thickness 0.15)
+				)
+			)
+		)
+		(pad "" np_thru_hole circle
+			(at 0 0)
+			(size 3.2 3.2)
+			(drill 3.2)
+			(layers "*.Cu" "*.Mask")
+		)
+		(embedded_fonts no)
+	)
 	(footprint "Resistor_THT:R_Axial_DIN0207_L6.3mm_D2.5mm_P10.16mm_Horizontal"
 		(layer "B.Cu")
@@
 		(layer "Edge.Cuts")
 	)
-	(gr_circle
-		(center 196.088 138.938)
-		(end 197.612 140.462)
-		(stroke
-			(width 0.05)
-			(type default)
-		)
-		(fill no)
-		(layer "Edge.Cuts")
-	)
 	(gr_line
 		(start 199.898 140.716)
@@
 		(layer "Edge.Cuts")
 	)
-	(gr_circle
-		(center 104.14 139.192)
-		(end 105.41 140.97)
-		(stroke
-			(width 0.05)
-			(type default)
-		)
-		(fill no)
-		(layer "Edge.Cuts")
-	)
 	(gr_line
 		(start 194.31 142.494)
@@
 			"ZjdSb0E2RzMwKzNnbVZzTkw2RHRXelBmMjloQUNRcG1BK1ZCMnJpMG5uUDhBeTFrSVBxeHFRRnMv"
 			"Tno5YSIKIkJNc1hOeEpkWERTeW5MTjI5S1lxbDIycnl4NHBFQmNnS09UWFJhYlpMYVFlYSszekQx"
-			"UHBRQmtMcFQ3QQ=="
+			"UHBRQmtMcFQ3Qd1SAwEAAADw0JNoAQAAAPB3CVgBAAAA0B5ZAwEAAADwdwlYAQAAAPB3CVgBAAAA"
+			"INGTaAEAAADwdwlYAQAAABAeWQMBAAAAUNGTaAEAAADwgUwDAQAAAICaWQMBAAAAQJtZAwEAAABQ"
+			"zVEDAQAAAPB3CVgBAAAA8HcJWAEAAADwdwlYAQAAAPCBTAMBAAAA8HcJWAEAAACA0ZNoAQAAAPB3"
+			"CVgBAAAA0B5ZAwEAAADwdwlYAQAAAPB3CVgBAAAAsNGTaAEAAACw41ADAQAAABAeWQMBAAAA4NGT"
+			"aAEAAACwdp9oAQAAAICaWQMBAAAAENKTaAEAAADwdwlYAQAAAECbWQMBAAAA8HcJWAEAAADwdwlY"
+			"AQAAAPB3CVgBAAAAUM1RAwEAAACw41ADAQAAALDjUAMBAAAAsONQAwEAAACwdp9oAQAAAPB3CVgB"
+			"AAAAsONQAwEAAABA0pNoAQAAAPB3CVgBAAAA0B5ZAwEAAADwdwlYAQAAAPB3CVgBAAAAcNKTaAEA"
+			"AACw41ADAQAAABAeWQMBAAAAoNKTaAEAAADwc59oAQAAAICaWQMBAAAA0NKTaAEAAAAwCU8DAQAA"
+			"ANAeWQMBAAAAMAlPAwEAAAAwCU8DAQAAADAJTwMBAAAAMAlPAwEAAAAA05NoAQAAAPB3CVgBAAAA"
+			"QJtZAwEAAADwdwlYAQAAADAJTwMBAAAAUM1RAwEAAACw41ADAQAAALDjUAMBAAAAsONQAwEAAADw"
+			"c59oAQAAADAJTwMBAAAAsONQAwEAAAAw05NoAQAAAPB3CVgBAAAA0B5ZAwEAAADwdwlYAQAAAPB3"
+			"CVgBAAAAYNOTaAEAAADwdwlYAQAAABAeWQMBAAAAkNOTaAEAAABw/0sDAQAAAICaWQMBAAAAwNOT"
+			"aAEAAACwOFYDAQAAABAeWQMBAAAAsDhWAwEAAADw05NoAQAAALB9swMBAAAA0AJaAwEAAACwOFYD"
+			"AQAAACDUk2gBAAAAsHYJWAEAAADgmlkDAQAAALB2CVgBAAAAsDhWAwEAAABQ1JNoAQAAAECbWQMB"
+			"AAAAsPxUAwEAAABQzVEDAQAAAPB3CVgBAAAA8HcJWAEAAADwdwlYAQAAAHD/SwMBAAAAsDhWAwEA"
+			"AADwdwlYAQAAAIDUk2gBAAAA8HcJWAEAAADQHlkDAQAAAPB3CVgBAAAA8HcJWAEAAACw1JNoAQAA"
+			"APB3CVgBAAAAEB5ZAwEAAADg1JNoAQAAAHD/SwMBAAAAgJpZAwEAAAAQ1ZNoAQAAALA4VgMBAAAA"
+			"EB5ZAwEAAACwOFYDAQAAAEDVk2gBAAAAsH2zAwEAAADgmlkDAQAAALA4VgMBAAAAsDhWAwEAAABw"
+			"1ZNoAQAAAECbWQ=="
 		)
 	)
-	(gr_text "Sord M5 Prototyping/ROM board\nleadedsolder.com v1 2025"
+	(gr_text "Sord M5 Prototyping/ROM board\nleadedsolder.com v2 2025"
 		(at 106.934 140.97 0)
 		(layer "F.SilkS")
